File: kicad/tentacle/pcb_octoprobe.kicad_sch (KiCad schematic)
At the start: 10 parts, among them J101 USB-226-BRW

Commit message: Tentacle v0.4
Parts:
- removed D102: LED_ERR (red), 00_project_library:LED_0603_1608Metric, symbol 00_project_library:LED GREEN
- removed R102: 1k, Resistor_SMD:R_0805_2012Metric, symbol Device:R
- added NT101, NT102, NT103, NT104, NT105, NT106: octoprobe_NetTie_USB_Differential, 00_project_library:octoprobe_NetTie_USB_Differential, symbol 00_project_library:octoprobe_NetTie_USB_Differential
- D101: value LED_BOOT (white) -> white; Label (none) -> LED_BOOT (white)
- D103: value LED_DUT_PWR (green) -> green; Label (none) -> LED_DUT_PWR (green)
- D104: value LED_INFRA_PWR (green) -> green; Label (none) -> LED_INFRA_PWR (green)
- R101: footprint Resistor_SMD:R_0603_1608Metric -> Resistor_SMD:R_0805_2012Metric
Connections:
- net USB Hub Chip/USB_DM2: now also NT103.3
- net USB Hub Chip/USB_DP2: now also NT103.1
- net USB3_DM: no longer names the net of J101.2 (D-)
- net USB3_DM: now also NT106.3
- net USB3_DP: no longer names the net of J101.3 (D+)
- net USB3_DP: now also NT106.1
- new net USB Hub Chip/USB_DM1: NT101.3
- new net USB Hub Chip/USB_DM3: NT105.1
- new net USB Hub Chip/USB_DP1: NT101.1
- new net USB Hub Chip/USB_DP3: NT105.3
- new net USB_DUT_D+: NT105.2, NT106.4
- new net USB_DUT_D-: NT105.4, NT106.2
- new net USB_INFRA_D+: NT103.2, NT104.4
- new net USB_INFRA_D-: NT103.4, NT104.2
- new net USB_PROBE_D+: NT101.2, NT102.4
- new net USB_PROBE_D-: NT101.4, NT102.2
- new net _USB_INFRA_D+: NT104.3
- new net _USB_INFRA_D-: NT104.1
- new net _USB_PROBE_D+: NT102.3
- new net _USB_PROBE_D-: NT102.1
- no-connect marks 4 -> 3
Other:
- added sheet RP2 PROBE (pcb_octoprobe_probe.kicad_sch)
- sheet RP2 CPU ports: added 12MHz; removed none
- note added: "Port 1: Probe - RP2"
- note added: "Port 2: Infra - RP2"
- note added: "Port 4: Infra - RP2 BOOT"
- note removed: "Port 1: Infra - RP2 PWR"
- note removed: "Port 2: Infra - RP2 BOOT"
- note removed: "Port 4: LED ERR"
- moved on the sheet: J101
