File: kicad/tentacle/pcb_octoprobe_cpu.kicad_sch (KiCad schematic)
At the start: 39 parts, among them J201 BOOT Button, Q201 NMOS, Q202 NMOS, SW201 RESET, U201 RP2040, U202 AMS1117-3.3, U203 W25Q128JVS, X201 Oscillator-12MHz

Commit message: Tentacle v0.4
Parts:
- removed BP201: GPIO9, 00_project_library:octoprobe_breakout_label, symbol 00_project_library:octoprobe_breakout_label
- removed BP202: GPIO10, 00_project_library:octoprobe_breakout_label, symbol 00_project_library:octoprobe_breakout_label
- removed BP203: GPIO11, 00_project_library:octoprobe_breakout_label, symbol 00_project_library:octoprobe_breakout_label
- removed BP204: GPIO12, 00_project_library:octoprobe_breakout_label, symbol 00_project_library:octoprobe_breakout_label
- removed BP205: GPIO13, 00_project_library:octoprobe_breakout_label, symbol 00_project_library:octoprobe_breakout_label
- removed BP206: GPIO14, 00_project_library:octoprobe_breakout_label, symbol 00_project_library:octoprobe_breakout_label
- removed BP207: GPIO15, 00_project_library:octoprobe_breakout_label, symbol 00_project_library:octoprobe_breakout_label
- removed J201: BOOT Button, Connector_PinHeader_2.54mm:PinHeader_1x02_P2.54mm_Vertical, symbol Connector:Conn_01x02_Pin
- removed Q201, Q202: NMOS, 00_project_library:SOT-23, symbol 00_project_library:NMOS
- removed R206: 0R, Resistor_SMD:R_0805_2012Metric, symbol Device:R
- removed R208: 1K, Resistor_SMD:R_0402_1005Metric, symbol Device:R
- removed SW201: RESET, 00_project_library:SW_TS-1187A-B-A-B, symbol 00_project_library:SW_MEC_5E
- added D203: red, 00_project_library:LED_0603_1608Metric, symbol 00_project_library:LED GREEN
- added J201: Conn_02x05, 00_project_library:PinSocket_2x05_P2.54mm_Vertical_squarepad, symbol Connector_Generic:Conn_02x05_Odd_Even
- C201, C202: JLC (none) -> C19702
- C203, C204, C207, C208, C209, C210, C211, C212, C213, C214: JLC (none) -> C1525
- C205, C206: JLC (none) -> C52923
- D201: value LED_ACTIVE (blue) -> blue; Label (none) -> LED_ACTIVE (blue)
- R204: value 10K -> 1k; now fitted
- U203: value W25Q128JVS -> W25Q32JVS; symbol 00_project_library:W25Q128JVS -> 00_project_library:W25Q32JVS; JCL C97521 -> (none); JLC C97521 -> C179173
Connections:
- net +3V3: no longer R204.1
- net +5V: now also J201.10 (Pin_10), J201.9 (Pin_9)
- net GND: now also D203.1 (K)
- net RELAIS_1: now also U201.11 (GPIO8); no longer U201.3 (GPIO1)
- net RELAIS_2: now also U201.12 (GPIO9); no longer U201.4 (GPIO2)
- net RELAIS_3: now also U201.13 (GPIO10); no longer U201.5 (GPIO3)
- net RELAIS_4: now also U201.14 (GPIO11); no longer U201.6 (GPIO4)
- net RELAIS_5: now also U201.15 (GPIO12); no longer U201.7 (GPIO5)
- net RELAIS_6: now also U201.16 (GPIO13); no longer U201.8 (GPIO6)
- net RELAIS_7: now also U201.17 (GPIO14); no longer U201.9 (GPIO7)
- net at R204.2: now also U201.18 (GPIO15)
- net at U201.2 (GPIO0): now also J201.1 (Pin_1)
- net RP2-USB-DM renamed _USB_INFRA_D-
- net RP2-USB-DP renamed _USB_INFRA_D+
- net XIN renamed 12MHz
- new net: J201.2 (Pin_2), U201.3 (GPIO1)
- new net: J201.3 (Pin_3), U201.4 (GPIO2)
- new net: J201.4 (Pin_4), U201.5 (GPIO3)
- new net: J201.5 (Pin_5), U201.6 (GPIO4)
- new net: J201.6 (Pin_6), U201.7 (GPIO5)
- new net: J201.7 (Pin_7), U201.8 (GPIO6)
- new net: J201.8 (Pin_8), U201.9 (GPIO7)
- new net: D203.2 (A), R204.1
- no-connect marks 18 -> 17
Other:
- note removed: "Boot: FET"
