File: kicad/tentacle/pcb_octoprobe_opto_relay.kicad_sch (KiCad schematic)
At the start: 5 parts, among them U1101 GAQY221S

Commit message: Tentacle v0.4
Parts:
- D1101: value LED WHITE -> white; Label (none) -> LED_RELAYS (white)
Changed lines of the file:
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@@
 		(shape output)
 		(at 111.76 69.85 0)
-		(fields_autoplaced yes)
 		(effects
 			(font
@@
 		(shape output)
 		(at 111.76 64.77 0)
-		(fields_autoplaced yes)
 		(effects
 			(font
@@
 		(shape input)
 		(at 60.96 49.53 180)
-		(fields_autoplaced yes)
 		(effects
 			(font
@@
 			)
 		)
-		(property "Value" "LED WHITE"
-			(at 101.9175 45.085 0)
+		(property "Value" "white"
+			(at 101.9175 44.45 0)
 			(effects
 				(font
@@
 			(at 100.33 49.53 0)
 			(effects
+				(font
+					(size 1.27 1.27)
+				)
+				(hide yes)
+			)
+		)
+		(property "Label" "LED_RELAYS (white)"
+			(at 100.33 49.53 0)
+			(effects
