File: kicad/tentacle/pcb_octoprobe_usbpowerswitch.kicad_sch (KiCad schematic)
At the start: 4 parts, among them U1401 MT9700

Commit message: Tentacle v0.4
Parts:
- C1401, C1402: JLC (none) -> C19702
- R1401: footprint Resistor_SMD:R_0805_2012Metric -> Resistor_SMD:R_0402_1005Metric
Changed lines of the file:
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@@
 		(shape input)
 		(at 81.28 81.28 180)
-		(fields_autoplaced yes)
 		(effects
 			(font
@@
 		(shape output)
 		(at 137.16 81.28 0)
-		(fields_autoplaced yes)
 		(effects
 			(font
@@
 			)
 		)
+		(property "JLC" "C19702"
+			(at -0.0001 177.8001 0)
+			(effects
+				(font
+					(size 1.27 1.27)
+				)
+				(hide yes)
+			)
+		)
+		(property "JLC" "C19702"
+			(at -0.0001 177.8001 0)
+			(effects
+				(font
+					(size 1.27 1.27)
+				)
+				(hide yes)
+			)
+		)
 		(pin "1"
 		)
@@
 					(unit 1)
 				)
-				(path "/35c47459-45a7-4753-acae-c8b47e7575e1/9cc2153c-44b9-4e7f-8961-835664992a07"
+				(path "/35c47459-45a7-4753-acae-c8b47e7575e1/d5925032-1cd4-4041-8ae3-121df5f0e5b4"
 					(reference "C402")
 					(unit 1)
@@
 					(unit 1)
 				)
-				(path "/35c47459-45a7-4753-acae-c8b47e7575e1/9cc2153c-44b9-4e7f-8961-835664992a07"
+				(path "/35c47459-45a7-4753-acae-c8b47e7575e1/d5925032-1cd4-4041-8ae3-121df5f0e5b4"
 					(reference "#PWR0404")
 					(unit 1)
@@
 					(unit 1)
 				)
-				(path "/35c47459-45a7-4753-acae-c8b47e7575e1/9cc2153c-44b9-4e7f-8961-835664992a07"
+				(path "/35c47459-45a7-4753-acae-c8b47e7575e1/d5925032-1cd4-4041-8ae3-121df5f0e5b4"
 					(reference "#SYM401")
 					(unit 1)
@@
 					(unit 1)
 				)
-				(path "/35c47459-45a7-4753-acae-c8b47e7575e1/9cc2153c-44b9-4e7f-8961-835664992a07"
+				(path "/35c47459-45a7-4753-acae-c8b47e7575e1/d5925032-1cd4-4041-8ae3-121df5f0e5b4"
 					(reference "#PWR0402")
 					(unit 1)
@@
 					(unit 1)
 				)
-				(path "/35c47459-45a7-4753-acae-c8b47e7575e1/9cc2153c-44b9-4e7f-8961-835664992a07"
+				(path "/35c47459-45a7-4753-acae-c8b47e7575e1/d5925032-1cd4-4041-8ae3-121df5f0e5b4"
 					(reference "#PWR0401")
 					(unit 1)
@@
 					(unit 1)
 				)
-				(path "/35c47459-45a7-4753-acae-c8b47e7575e1/9cc2153c-44b9-4e7f-8961-835664992a07"
+				(path "/35c47459-45a7-4753-acae-c8b47e7575e1/d5925032-1cd4-4041-8ae3-121df5f0e5b4"
 					(reference "#PWR0403")
 					(unit 1)
@@
 					(unit 1)
 				)
-				(path "/35c47459-45a7-4753-acae-c8b47e7575e1/9cc2153c-44b9-4e7f-8961-835664992a07"
+				(path "/35c47459-45a7-4753-acae-c8b47e7575e1/d5925032-1cd4-4041-8ae3-121df5f0e5b4"
 					(reference "U401")
 					(unit 1)
@@
 					(unit 1)
 				)
-				(path "/35c47459-45a7-4753-acae-c8b47e7575e1/9cc2153c-44b9-4e7f-8961-835664992a07"
+				(path "/35c47459-45a7-4753-acae-c8b47e7575e1/d5925032-1cd4-4041-8ae3-121df5f0e5b4"
 					(reference "#PWR0405")
 					(unit 1)
@@
 			)
 		)
+		(property "JLC" "C19702"
+			(at 180.3401 -0.0001 0)
+			(effects
+				(font
+					(size 1.27 1.27)
+				)
+				(hide yes)
+			)
+		)
+		(property "JLC" "C19702"
+			(at 180.3401 -0.0001 0)
+			(effects
+				(font
+					(size 1.27 1.27)
+				)
+				(hide yes)
+			)
+		)
 		(pin "1"
 		)
@@
 					(unit 1)
 				)
-				(path "/35c47459-45a7-4753-acae-c8b47e7575e1/9cc2153c-44b9-4e7f-8961-835664992a07"
+				(path "/35c47459-45a7-4753-acae-c8b47e7575e1/d5925032-1cd4-4041-8ae3-121df5f0e5b4"
 					(reference "C401")
 					(unit 1)
@@
 			)
 		)
-		(property "Footprint" "Resistor_SMD:R_0805_2012Metric"
+		(property "Footprint" "Resistor_SMD:R_0402_1005Metric"
 			(at 81.788 90.17 90)
 			(effects
@@
 					(unit 1)
 				)
-				(path "/35c47459-45a7-4753-acae-c8b47e7575e1/9cc2153c-44b9-4e7f-8961-835664992a07"
+				(path "/35c47459-45a7-4753-acae-c8b47e7575e1/d5925032-1cd4-4041-8ae3-121df5f0e5b4"
 					(reference "R401")
 					(unit 1)
