File: kicad/tentacle/pcb_octoprobe.kicad_pcb (KiCad board)
At the start: 2 copper layers, 100 x 160 mm, 660 parts, among them J101 USB-226-BRW, J1301 Conn_01x20, J1302 Conn_01x20, J1303 Conn_01x20, J201 BOOT Button, J301 USB_C_Receptacle_USB2.0, J501 Conn_01x20, J502 Conn_01x20, Q201 NMOS, Q202 NMOS, SW201 RESET, U1001 GAQY221S, U1101 GAQY221S, U1201 GAQY221S, U1401 MT9700, U201 RP2040, U202 AMS1117-3.3, U203 W25Q128JVS, U301 AMS1117-3.3, U302 USB2514B_Bi, U401 MT9700, U601 GAQY221S, U701 GAQY221S, U801 GAQY221S, U901 GAQY221S, X201 Oscillator-12MHz, Y301 24MHz

Commit message: Tentacle v0.4
Parts:
- removed the BP1301 at (81.6, 121.4)
- removed the BP1301 at (79.1, 134.1)
- removed the BP1301 at (81.6, 136.6)
- removed the BP1301 at (96.9, 167.1)
- removed the BP1301 at (114.6, 164.6)
- removed the BP1301 at (124.8, 167.1)
- removed the BP1301 at (81.6, 167.1)
- removed the BP1301 at (81.6, 134.1)
- removed the BP1301 at (86.7, 164.6)
- removed the BP1301 at (81.6, 157.0)
- removed the BP1301 at (142.6, 167.1)
- removed the BP1301 at (94.3, 164.6)
- removed the BP1301 at (122.3, 164.6)
- removed the BP1301 at (84.2, 167.1)
- removed the BP1301 at (119.7, 167.1)
- removed the BP1301 at (81.6, 126.5)
- removed the BP1301 at (81.6, 151.9)
- removed the BP1301 at (107.0, 167.1)
- removed the BP1301 at (140.0, 167.1)
- removed the BP1301 at (84.2, 164.6)
- removed the BP1301 at (142.6, 164.6)
- removed the BP1301 at (79.1, 123.9)
- removed the BP1301 at (79.1, 144.3)
- removed the BP1301 at (91.8, 167.1)
- removed the BP1301 at (79.1, 167.1)
- removed the BP1301 at (101.9, 167.1)
- removed the BP1301 at (129.9, 167.1)
- removed the BP1301 at (129.9, 164.6)
- removed the BP1301 at (135.0, 167.1)
- removed the BP1301 at (122.3, 167.1)
- removed the BP1301 at (81.6, 123.9)
- removed the BP1301 at (127.3, 164.6)
- removed the BP1301 at (81.6, 164.6)
- removed the BP1301 at (79.1, 159.5)
- removed the BP1301 at (81.6, 144.3)
- removed the BP1301 at (114.6, 167.1)
- removed the BP1301 at (81.6, 129.0)
- removed the BP1301 at (109.6, 167.1)
- removed the BP1301 at (127.3, 167.1)
- removed the BP1301 at (79.1, 131.6)
- removed the BP1301 at (79.1, 129.0)
- removed the BP1301 at (119.7, 164.6)
- removed the BP1301 at (79.1, 139.2)
- removed the BP1301 at (137.5, 164.6)
- removed the BP1301 at (81.6, 131.6)
- removed the BP1301 at (135.0, 164.6)
- removed the BP1301 at (89.2, 164.6)
- removed the BP1301 at (79.1, 118.9)
- removed the BP1301 at (79.1, 149.3)
- removed the BP1301 at (86.7, 167.1)
- removed the BP1301 at (79.1, 141.7)
- removed the BP1301 at (91.8, 164.6)
- removed the BP1301 at (117.2, 167.1)
- removed the BP1301 at (81.6, 139.2)
- removed the BP1301 at (81.6, 146.8)
- removed the BP1301 at (117.2, 164.6)
- removed the BP1301 at (99.4, 164.6)
- removed the BP1301 at (81.6, 118.9)
- removed the BP1301 at (81.6, 141.7)
- removed the BP1301 at (79.1, 164.6)
- removed the BP1301 at (112.1, 167.1)
- removed the BP1301 at (79.1, 126.5)
- removed the BP1301 at (132.4, 167.1)
- removed the BP1301 at (81.6, 149.3)
- removed the BP1301 at (81.6, 159.5)
- removed the BP1301 at (94.3, 167.1)
- removed the BP1301 at (132.4, 164.6)
- removed the BP1301 at (124.8, 164.6)
- removed the BP1301 at (96.9, 164.6)
- removed the BP1301 at (79.1, 154.4)
- removed the BP1301 at (79.1, 146.8)
- removed the BP1301 at (79.1, 162.0)
- removed the BP1301 at (101.9, 164.6)
- removed the BP1301 at (112.1, 164.6)
- removed the BP1301 at (104.5, 164.6)
- removed the BP1301 at (99.4, 167.1)
- removed the BP1301 at (109.6, 164.6)
- removed the BP1301 at (79.1, 121.4)
- removed the BP1301 at (81.6, 154.4)
- removed the BP1301 at (79.1, 151.9)
- removed the BP1301 at (79.1, 136.6)
- removed the BP1301 at (89.2, 167.1)
- removed the BP1301 at (79.1, 157.0)
- removed the BP1301 at (81.6, 162.0)
- removed the BP1301 at (140.0, 164.6)
- removed the BP1301 at (107.0, 164.6)
- removed the BP1301 at (104.5, 167.1)
- removed the BP1301 at (137.5, 167.1)
- removed BP201: GPIO9, 00_project_library:octoprobe_breakout_label
- removed BP202: GPIO10, 00_project_library:octoprobe_breakout_label
- removed BP203: GPIO11, 00_project_library:octoprobe_breakout_label
- removed BP204: GPIO12, 00_project_library:octoprobe_breakout_label
- removed BP205: GPIO13, 00_project_library:octoprobe_breakout_label
- removed BP206: GPIO14, 00_project_library:octoprobe_breakout_label
- removed BP207: GPIO15, 00_project_library:octoprobe_breakout_label
- removed D102: LED_ERR (red), 00_project_library:LED_0603_1608Metric
- removed J1301: Conn_01x20, 00_project_library:PinSocket_2x20_P2.54mm_Vertical-stackable_squarepad
- removed J502: Conn_01x20, 00_project_library:PinSocket_2x20_P2.54mm_Vertical_squarepad
- removed Q201, Q202: NMOS, 00_project_library:SOT-23
- removed R102: 1k, Resistor_SMD:R_0805_2012Metric
- removed R206: 0R, Resistor_SMD:R_0805_2012Metric
- removed R208: 1K, Resistor_SMD:R_0402_1005Metric
- removed SW201: RESET, 00_project_library:SW_TS-1187A-B-A-B
- added BP1301: prototype_GND, 00_project_library:octoprobe_breakout_PB, F.Cu at (74.0, 103.6)
- added BP1301: prototype_GND, 00_project_library:octoprobe_breakout_PB, F.Cu at (74.0, 106.2)
- added BP1301: prototype_GND, 00_project_library:octoprobe_breakout_PB, F.Cu at (68.9, 106.2)
- added BP1301: prototype_GND, 00_project_library:octoprobe_breakout_PB, F.Cu at (63.8, 103.6)
- added BP1301: prototype_GND, 00_project_library:octoprobe_breakout_PB, F.Cu at (66.4, 103.6)
- added BP1301: prototype_GND, 00_project_library:octoprobe_breakout_PB, F.Cu at (135.0, 149.3)
- added BP1301: prototype_GND, 00_project_library:octoprobe_breakout_PB, F.Cu at (135.0, 151.9)
- added BP1301: prototype_GND, 00_project_library:octoprobe_breakout_PB, F.Cu at (66.4, 106.2)
- added BP1301: prototype_GND, 00_project_library:octoprobe_breakout_PB, F.Cu at (63.8, 106.2)
- added BP1301: prototype_GND, 00_project_library:octoprobe_breakout_PB, F.Cu at (132.4, 151.9)
- added BP1301: prototype_GND, 00_project_library:octoprobe_breakout_PB, F.Cu at (71.5, 103.6)
- added BP1301: prototype_GND, 00_project_library:octoprobe_breakout_PB, F.Cu at (132.4, 149.3)
- added BP1301: prototype_GND, 00_project_library:octoprobe_breakout_PB, F.Cu at (68.9, 103.6)
- added BP1301: prototype_GND, 00_project_library:octoprobe_breakout_PB, F.Cu at (71.5, 106.2)
- added BP1302: prototype_NC, 00_project_library:octoprobe_breakout_PB_NC, F.Cu at (114.6, 149.3)
- added BP1302: prototype_NC, 00_project_library:octoprobe_breakout_PB_NC, F.Cu at (63.8, 151.9)
- added BP1302: prototype_NC, 00_project_library:octoprobe_breakout_PB_NC, F.Cu at (94.3, 149.3)
- added BP1302: prototype_NC, 00_project_library:octoprobe_breakout_PB_NC, F.Cu at (89.2, 149.3)
- added BP1302: prototype_NC, 00_project_library:octoprobe_breakout_PB_NC, F.Cu at (127.3, 151.9)
- added BP1302: prototype_NC, 00_project_library:octoprobe_breakout_PB_NC, F.Cu at (66.4, 144.3)
- added BP1302: prototype_NC, 00_project_library:octoprobe_breakout_PB_NC, F.Cu at (68.9, 144.3)
- added BP1302: prototype_NC, 00_project_library:octoprobe_breakout_PB_NC, F.Cu at (109.6, 149.3)
- added BP1302: prototype_NC, 00_project_library:octoprobe_breakout_PB_NC, F.Cu at (79.1, 151.9)
- added BP1302: prototype_NC, 00_project_library:octoprobe_breakout_PB_NC, F.Cu at (89.2, 151.9)
- added BP1302: prototype_NC, 00_project_library:octoprobe_breakout_PB_NC, F.Cu at (96.9, 151.9)
- added BP1302: prototype_NC, 00_project_library:octoprobe_breakout_PB_NC, F.Cu at (71.5, 116.3)
- added BP1302: prototype_NC, 00_project_library:octoprobe_breakout_PB_NC, F.Cu at (63.8, 111.2)
- added BP1302: prototype_NC, 00_project_library:octoprobe_breakout_PB_NC, F.Cu at (117.2, 149.3)
- added BP1302: prototype_NC, 00_project_library:octoprobe_breakout_PB_NC, F.Cu at (63.8, 113.8)
- added BP1302: prototype_NC, 00_project_library:octoprobe_breakout_PB_NC, F.Cu at (129.9, 149.3)
- added BP1302: prototype_NC, 00_project_library:octoprobe_breakout_PB_NC, F.Cu at (68.9, 108.7)
- added BP1302: prototype_NC, 00_project_library:octoprobe_breakout_PB_NC, F.Cu at (68.9, 123.9)
- added BP1302: prototype_NC, 00_project_library:octoprobe_breakout_PB_NC, F.Cu at (74.0, 111.2)
- added BP1302: prototype_NC, 00_project_library:octoprobe_breakout_PB_NC, F.Cu at (68.9, 126.5)
- added BP1302: prototype_NC, 00_project_library:octoprobe_breakout_PB_NC, F.Cu at (68.9, 131.6)
- added BP1302: prototype_NC, 00_project_library:octoprobe_breakout_PB_NC, F.Cu at (66.4, 123.9)
- added BP1302: prototype_NC, 00_project_library:octoprobe_breakout_PB_NC, F.Cu at (74.0, 129.0)
- added BP1302: prototype_NC, 00_project_library:octoprobe_breakout_PB_NC, F.Cu at (63.8, 118.9)
- added BP1302: prototype_NC, 00_project_library:octoprobe_breakout_PB_NC, F.Cu at (63.8, 134.1)
- added BP1302: prototype_NC, 00_project_library:octoprobe_breakout_PB_NC, F.Cu at (66.4, 118.9)
- added BP1302: prototype_NC, 00_project_library:octoprobe_breakout_PB_NC, F.Cu at (101.9, 149.3)
- added BP1302: prototype_NC, 00_project_library:octoprobe_breakout_PB_NC, F.Cu at (74.0, 139.2)
- added BP1302: prototype_NC, 00_project_library:octoprobe_breakout_PB_NC, F.Cu at (112.1, 151.9)
- added BP1302: prototype_NC, 00_project_library:octoprobe_breakout_PB_NC, F.Cu at (63.8, 146.8)
- added BP1302: prototype_NC, 00_project_library:octoprobe_breakout_PB_NC, F.Cu at (107.0, 151.9)
- added BP1302: prototype_NC, 00_project_library:octoprobe_breakout_PB_NC, F.Cu at (68.9, 118.9)
- added BP1302: prototype_NC, 00_project_library:octoprobe_breakout_PB_NC, F.Cu at (68.9, 113.8)
- added BP1302: prototype_NC, 00_project_library:octoprobe_breakout_PB_NC, F.Cu at (71.5, 144.3)
- added BP1302: prototype_NC, 00_project_library:octoprobe_breakout_PB_NC, F.Cu at (104.5, 149.3)
- added BP1302: prototype_NC, 00_project_library:octoprobe_breakout_PB_NC, F.Cu at (71.5, 126.5)
- added BP1302: prototype_NC, 00_project_library:octoprobe_breakout_PB_NC, F.Cu at (68.9, 136.6)
- added BP1302: prototype_NC, 00_project_library:octoprobe_breakout_PB_NC, F.Cu at (74.0, 113.8)
- added BP1302: prototype_NC, 00_project_library:octoprobe_breakout_PB_NC, F.Cu at (68.9, 139.2)
- added BP1302: prototype_NC, 00_project_library:octoprobe_breakout_PB_NC, F.Cu at (74.0, 131.6)
- added BP1302: prototype_NC, 00_project_library:octoprobe_breakout_PB_NC, F.Cu at (74.0, 136.6)
- added BP1302: prototype_NC, 00_project_library:octoprobe_breakout_PB_NC, F.Cu at (68.9, 134.1)
- added BP1302: prototype_NC, 00_project_library:octoprobe_breakout_PB_NC, F.Cu at (124.8, 149.3)
- added BP1302: prototype_NC, 00_project_library:octoprobe_breakout_PB_NC, F.Cu at (71.5, 151.9)
- added BP1302: prototype_NC, 00_project_library:octoprobe_breakout_PB_NC, F.Cu at (91.8, 149.3)
- added BP1302: prototype_NC, 00_project_library:octoprobe_breakout_PB_NC, F.Cu at (96.9, 149.3)
- added BP1302: prototype_NC, 00_project_library:octoprobe_breakout_PB_NC, F.Cu at (66.4, 146.8)
- added BP1302: prototype_NC, 00_project_library:octoprobe_breakout_PB_NC, F.Cu at (109.6, 151.9)
- added BP1302: prototype_NC, 00_project_library:octoprobe_breakout_PB_NC, F.Cu at (74.0, 146.8)
- added BP1302: prototype_NC, 00_project_library:octoprobe_breakout_PB_NC, F.Cu at (91.8, 151.9)
- added BP1302: prototype_NC, 00_project_library:octoprobe_breakout_PB_NC, F.Cu at (63.8, 141.7)
- added BP1302: prototype_NC, 00_project_library:octoprobe_breakout_PB_NC, F.Cu at (66.4, 151.9)
- added BP1302: prototype_NC, 00_project_library:octoprobe_breakout_PB_NC, F.Cu at (63.8, 131.6)
- added BP1302: prototype_NC, 00_project_library:octoprobe_breakout_PB_NC, F.Cu at (63.8, 126.5)
- added BP1302: prototype_NC, 00_project_library:octoprobe_breakout_PB_NC, F.Cu at (99.4, 151.9)
- added BP1302: prototype_NC, 00_project_library:octoprobe_breakout_PB_NC, F.Cu at (117.2, 151.9)
- added BP1302: prototype_NC, 00_project_library:octoprobe_breakout_PB_NC, F.Cu at (74.0, 123.9)
- added BP1302: prototype_NC, 00_project_library:octoprobe_breakout_PB_NC, F.Cu at (63.8, 123.9)
- added BP1302: prototype_NC, 00_project_library:octoprobe_breakout_PB_NC, F.Cu at (76.5, 151.9)
- added BP1302: prototype_NC, 00_project_library:octoprobe_breakout_PB_NC, F.Cu at (71.5, 141.7)
- added BP1302: prototype_NC, 00_project_library:octoprobe_breakout_PB_NC, F.Cu at (71.5, 136.6)
- added BP1302: prototype_NC, 00_project_library:octoprobe_breakout_PB_NC, F.Cu at (74.0, 151.9)
- added BP1302: prototype_NC, 00_project_library:octoprobe_breakout_PB_NC, F.Cu at (68.9, 149.3)
- added BP1302: prototype_NC, 00_project_library:octoprobe_breakout_PB_NC, F.Cu at (119.7, 151.9)
- added BP1302: prototype_NC, 00_project_library:octoprobe_breakout_PB_NC, F.Cu at (127.3, 149.3)
- added BP1302: prototype_NC, 00_project_library:octoprobe_breakout_PB_NC, F.Cu at (101.9, 151.9)
- added BP1302: prototype_NC, 00_project_library:octoprobe_breakout_PB_NC, F.Cu at (68.9, 151.9)
- added BP1302: prototype_NC, 00_project_library:octoprobe_breakout_PB_NC, F.Cu at (74.0, 134.1)
- added BP1302: prototype_NC, 00_project_library:octoprobe_breakout_PB_NC, F.Cu at (71.5, 139.2)
- added BP1302: prototype_NC, 00_project_library:octoprobe_breakout_PB_NC, F.Cu at (74.0, 149.3)
- added BP1302: prototype_NC, 00_project_library:octoprobe_breakout_PB_NC, F.Cu at (81.6, 151.9)
- added BP1302: prototype_NC, 00_project_library:octoprobe_breakout_PB_NC, F.Cu at (63.8, 129.0)
- added BP1302: prototype_NC, 00_project_library:octoprobe_breakout_PB_NC, F.Cu at (74.0, 118.9)
- added BP1302: prototype_NC, 00_project_library:octoprobe_breakout_PB_NC, F.Cu at (86.7, 149.3)
- added BP1302: prototype_NC, 00_project_library:octoprobe_breakout_PB_NC, F.Cu at (63.8, 139.2)
- added BP1302: prototype_NC, 00_project_library:octoprobe_breakout_PB_NC, F.Cu at (66.4, 129.0)
- added BP1302: prototype_NC, 00_project_library:octoprobe_breakout_PB_NC, F.Cu at (114.6, 151.9)
- added BP1302: prototype_NC, 00_project_library:octoprobe_breakout_PB_NC, F.Cu at (66.4, 141.7)
- added BP1302: prototype_NC, 00_project_library:octoprobe_breakout_PB_NC, F.Cu at (66.4, 139.2)
- added BP1302: prototype_NC, 00_project_library:octoprobe_breakout_PB_NC, F.Cu at (66.4, 134.1)
- added BP1302: prototype_NC, 00_project_library:octoprobe_breakout_PB_NC, F.Cu at (112.1, 149.3)
- added BP1302: prototype_NC, 00_project_library:octoprobe_breakout_PB_NC, F.Cu at (71.5, 118.9)
- added BP1302: prototype_NC, 00_project_library:octoprobe_breakout_PB_NC, F.Cu at (68.9, 146.8)
- added BP1302: prototype_NC, 00_project_library:octoprobe_breakout_PB_NC, F.Cu at (68.9, 121.4)
- added BP1302: prototype_NC, 00_project_library:octoprobe_breakout_PB_NC, F.Cu at (68.9, 129.0)
- added BP1302: prototype_NC, 00_project_library:octoprobe_breakout_PB_NC, F.Cu at (63.8, 116.3)
- added BP1302: prototype_NC, 00_project_library:octoprobe_breakout_PB_NC, F.Cu at (71.5, 131.6)
- added BP1302: prototype_NC, 00_project_library:octoprobe_breakout_PB_NC, F.Cu at (63.8, 136.6)
- added BP1302: prototype_NC, 00_project_library:octoprobe_breakout_PB_NC, F.Cu at (99.4, 149.3)
- added BP1302: prototype_NC, 00_project_library:octoprobe_breakout_PB_NC, F.Cu at (119.7, 149.3)
- added BP1302: prototype_NC, 00_project_library:octoprobe_breakout_PB_NC, F.Cu at (71.5, 123.9)
- added BP1302: prototype_NC, 00_project_library:octoprobe_breakout_PB_NC, F.Cu at (79.1, 149.3)
- added BP1302: prototype_NC, 00_project_library:octoprobe_breakout_PB_NC, F.Cu at (66.4, 111.2)
- added BP1302: prototype_NC, 00_project_library:octoprobe_breakout_PB_NC, F.Cu at (66.4, 131.6)
- added BP1302: prototype_NC, 00_project_library:octoprobe_breakout_PB_NC, F.Cu at (71.5, 129.0)
- added BP1302: prototype_NC, 00_project_library:octoprobe_breakout_PB_NC, F.Cu at (66.4, 149.3)
- added BP1302: prototype_NC, 00_project_library:octoprobe_breakout_PB_NC, F.Cu at (68.9, 111.2)
- added BP1302: prototype_NC, 00_project_library:octoprobe_breakout_PB_NC, F.Cu at (66.4, 121.4)
- added BP1302: prototype_NC, 00_project_library:octoprobe_breakout_PB_NC, F.Cu at (71.5, 149.3)
- added BP1302: prototype_NC, 00_project_library:octoprobe_breakout_PB_NC, F.Cu at (129.9, 151.9)
- added BP1302: prototype_NC, 00_project_library:octoprobe_breakout_PB_NC, F.Cu at (94.3, 151.9)
- added BP1302: prototype_NC, 00_project_library:octoprobe_breakout_PB_NC, F.Cu at (84.2, 151.9)
- added BP1302: prototype_NC, 00_project_library:octoprobe_breakout_PB_NC, F.Cu at (63.8, 144.3)
- added BP1302: prototype_NC, 00_project_library:octoprobe_breakout_PB_NC, F.Cu at (76.5, 149.3)
- added BP1302: prototype_NC, 00_project_library:octoprobe_breakout_PB_NC, F.Cu at (68.9, 141.7)
- added BP1302: prototype_NC, 00_project_library:octoprobe_breakout_PB_NC, F.Cu at (63.8, 121.4)
- added BP1302: prototype_NC, 00_project_library:octoprobe_breakout_PB_NC, F.Cu at (66.4, 126.5)
- added BP1302: prototype_NC, 00_project_library:octoprobe_breakout_PB_NC, F.Cu at (74.0, 141.7)
- added BP1302: prototype_NC, 00_project_library:octoprobe_breakout_PB_NC, F.Cu at (74.0, 116.3)
- added BP1302: prototype_NC, 00_project_library:octoprobe_breakout_PB_NC, F.Cu at (66.4, 116.3)
- added BP1302: prototype_NC, 00_project_library:octoprobe_breakout_PB_NC, F.Cu at (86.7, 151.9)
- added BP1302: prototype_NC, 00_project_library:octoprobe_breakout_PB_NC, F.Cu at (74.0, 121.4)
- added BP1302: prototype_NC, 00_project_library:octoprobe_breakout_PB_NC, F.Cu at (71.5, 146.8)
- added BP1302: prototype_NC, 00_project_library:octoprobe_breakout_PB_NC, F.Cu at (74.0, 126.5)
- added BP1302: prototype_NC, 00_project_library:octoprobe_breakout_PB_NC, F.Cu at (81.6, 149.3)
- added BP1302: prototype_NC, 00_project_library:octoprobe_breakout_PB_NC, F.Cu at (71.5, 111.2)
- added BP1302: prototype_NC, 00_project_library:octoprobe_breakout_PB_NC, F.Cu at (74.0, 108.7)
- added BP1302: prototype_NC, 00_project_library:octoprobe_breakout_PB_NC, F.Cu at (104.5, 151.9)
- added BP1302: prototype_NC, 00_project_library:octoprobe_breakout_PB_NC, F.Cu at (122.3, 151.9)
- added BP1302: prototype_NC, 00_project_library:octoprobe_breakout_PB_NC, F.Cu at (122.3, 149.3)
- added BP1302: prototype_NC, 00_project_library:octoprobe_breakout_PB_NC, F.Cu at (71.5, 108.7)
- added BP1302: prototype_NC, 00_project_library:octoprobe_breakout_PB_NC, F.Cu at (63.8, 149.3)
- added BP1302: prototype_NC, 00_project_library:octoprobe_breakout_PB_NC, F.Cu at (68.9, 116.3)
- added BP1302: prototype_NC, 00_project_library:octoprobe_breakout_PB_NC, F.Cu at (63.8, 108.7)
- added BP1302: prototype_NC, 00_project_library:octoprobe_breakout_PB_NC, F.Cu at (74.0, 144.3)
- added BP1302: prototype_NC, 00_project_library:octoprobe_breakout_PB_NC, F.Cu at (71.5, 113.8)
- added BP1302: prototype_NC, 00_project_library:octoprobe_breakout_PB_NC, F.Cu at (124.8, 151.9)
- added BP1302: prototype_NC, 00_project_library:octoprobe_breakout_PB_NC, F.Cu at (84.2, 149.3)
- added BP1302: prototype_NC, 00_project_library:octoprobe_breakout_PB_NC, F.Cu at (107.0, 149.3)
- added BP1302: prototype_NC, 00_project_library:octoprobe_breakout_PB_NC, F.Cu at (66.4, 113.8)
- added BP1302: prototype_NC, 00_project_library:octoprobe_breakout_PB_NC, F.Cu at (71.5, 134.1)
- added BP1302: prototype_NC, 00_project_library:octoprobe_breakout_PB_NC, F.Cu at (66.4, 108.7)
- added BP1302: prototype_NC, 00_project_library:octoprobe_breakout_PB_NC, F.Cu at (71.5, 121.4)
- added BP1302: prototype_NC, 00_project_library:octoprobe_breakout_PB_NC, F.Cu at (66.4, 136.6)
- added C1501: 100n, Capacitor_SMD:C_0402_1005Metric, F.Cu at (84.9, 46.6)
- added C1502: 100n, Capacitor_SMD:C_0402_1005Metric, F.Cu at (70.4, 48.2)
- added C1503: 1u, Capacitor_SMD:C_0402_1005Metric, F.Cu at (74.0, 44.6)
- added C1504: 1u, Capacitor_SMD:C_0402_1005Metric, F.Cu at (74.0, 43.6)
- added C1505: 100n, Capacitor_SMD:C_0402_1005Metric, F.Cu at (70.4, 47.3)
- added C1506: 100n, Capacitor_SMD:C_0402_1005Metric, F.Cu at (74.0, 42.7)
- added C1507: 100n, Capacitor_SMD:C_0402_1005Metric, F.Cu at (60.9, 45.5)
- added C1508: 100n, Capacitor_SMD:C_0402_1005Metric, F.Cu at (84.9, 47.5)
- added C1509: 100n, Capacitor_SMD:C_0402_1005Metric, F.Cu at (76.1, 52.9)
- added C1510: 100n, Capacitor_SMD:C_0402_1005Metric, F.Cu at (80.8, 43.0)
- added C1511: 100n, Capacitor_SMD:C_0402_1005Metric, F.Cu at (80.0, 53.4)
- added C1512: 100n, Capacitor_SMD:C_0402_1005Metric, F.Cu at (98.8, 31.1)
- added D1501: B5819W SL, Diode_SMD:D_SOD-123, F.Cu at (67.0, 58.4)
- added D203: red, 00_project_library:LED_0603_1608Metric, F.Cu at (121.3, 177.7)
- added J1501: Conn_02x20, 00_project_library:PinSocket_2x12_P2.54mm_Vertical_squarepad, F.Cu at (65.1, 66.0)
- added J1502: Conn_01x12, 00_project_library:PinSocket_1x12_P2.54mm_Vertical_squarepad, F.Cu at (65.1, 84.6)
- added Logo_open_hardware101: Logo_Open_Hardware_Small, Symbol:OSHW-Logo2_9.8x8mm_SilkScreen, B.Cu at (153.2, 50.3)
- added NT101: octoprobe_NetTie_USB_Differential, 00_project_library:octoprobe_NetTie_USB_Differential, F.Cu at (120.4, 34.4)
- added NT102: octoprobe_NetTie_USB_Differential, 00_project_library:octoprobe_NetTie_USB_Differential, F.Cu at (70.4, 43.3)
- added NT103: octoprobe_NetTie_USB_Differential, 00_project_library:octoprobe_NetTie_USB_Differential, F.Cu at (123.5, 35.2)
- added NT104: octoprobe_NetTie_USB_Differential, 00_project_library:octoprobe_NetTie_USB_Differential, F.Cu at (126.0, 44.2)
- added NT105: octoprobe_NetTie_USB_Differential, 00_project_library:octoprobe_NetTie_USB_Differential, F.Cu at (126.2, 34.2)
- added NT106: octoprobe_NetTie_USB_Differential, 00_project_library:octoprobe_NetTie_USB_Differential, F.Cu at (139.1, 33.0)
- added NT301: octoprobe_NetTie_USB_Differential, 00_project_library:octoprobe_NetTie_USB_Differential, F.Cu at (86.4, 18.4)
- added NT302: octoprobe_NetTie_USB_Differential, 00_project_library:octoprobe_NetTie_USB_Differential, F.Cu at (117.0, 23.3)
- added R1501: 27R, Resistor_SMD:R_0402_1005Metric, F.Cu at (70.8, 45.4)
- added R1502: 27R, Resistor_SMD:R_0402_1005Metric, F.Cu at (69.9, 45.4)
- added R1503: 0R, Resistor_SMD:R_0805_2012Metric, F.Cu at (62.9, 58.2)
- added R1504: 10K, Resistor_SMD:R_0402_1005Metric, F.Cu at (73.5, 51.1)
- added R1505: 100K, Resistor_SMD:R_0402_1005Metric, F.Cu at (67.9, 76.6)
- added U1501: RP2040, 00_project_library:RP2040-QFN-56, F.Cu at (79.1, 47.7)
- added U1502: W25Q32JVS, 00_project_library:SOIC-8_5.23x5.23mm_P1.27mm, F.Cu at (62.8, 51.8)
- added U1503: TXB0108PW, Package_SO:TSSOP-20_4.4x6.5mm_P0.65mm, F.Cu at (74.0, 77.5)
- D1001, D1101, D1201, D601, D701, D801, D901: value LED WHITE -> white
- D101: value LED_BOOT (white) -> white
- D103: value LED_DUT_PWR (green) -> green
- D104: value LED_INFRA_PWR (green) -> green
- D201: value LED_ACTIVE (blue) -> blue
- D301: value LED_PWR (green) -> green
- J1302, J1303: value Conn_01x20 -> Conn_02x20
- J201: value BOOT Button -> Conn_02x05; footprint Connector_PinHeader_2.54mm:PinHeader_1x02_P2.54mm_Vertical -> 00_project_library:PinSocket_2x05_P2.54mm_Vertical_squarepad
- J501: value Conn_01x20 -> Conn_02x20; footprint 00_project_library:PinSocket_2x20_P2.54mm_Vertical_squarepad -> 00_project_library:PinSocket_2x14_P2.54mm_Vertical_squarepad
- R101, R301: footprint Resistor_SMD:R_0603_1608Metric -> Resistor_SMD:R_0805_2012Metric
- R1401, R401: footprint Resistor_SMD:R_0805_2012Metric -> Resistor_SMD:R_0402_1005Metric
- R204: value 10K -> 1k
- U203: value W25Q128JVS -> W25Q32JVS
- moved R103 138.3 mm to (71.3, 177.9)
- moved R201 133.4 mm to (98.3, 177.9)
- moved R204 117.3 mm to (125.1, 177.7)
- moved D104 100.2 mm to (148.2, 177.9)
- moved R104 73.2 mm to (151.9, 177.9)
- moved D201 72.2 mm to (94.5, 177.9)
- moved D103 70.0 mm to (67.4, 177.9)
- moved C402 69.4 mm to (125.0, 19.0), turned to 180 degrees
- moved C401 67.5 mm to (84.7, 27.2), turned to 90 degrees
- moved D301 55.2 mm to (89.7, 22.1), turned to 0 degrees
- moved R302 55.1 mm to (81.9, 27.0)
- moved R303 55.1 mm to (78.7, 27.2)
- moved D302 55.1 mm to (80.2, 27.9), turned to -90 degrees
- moved J301 55.1 mm to (80.7, 22.2)
- moved C203 54.2 mm to (141.1, 46.6), turned to 0 degrees
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Connections:
- net +1V1 renamed /RP2 CPU/+1V1
- net /RP2 CPU/XIN renamed /RP2 CPU/12MHz
- D302 pad 1: /USB Hub Chip/USBDP -> Net-(D302-I/O1-Pad1)
- D302 pad 3: /USB Hub Chip/USBDM -> Net-(D302-I/O2-Pad3)
- D302 pad 4: /USB Hub Chip/USBDM -> Net-(D302-I/O2-Pad3)
- D302 pad 6: /USB Hub Chip/USBDP -> Net-(D302-I/O1-Pad1)
- J101 pad 2: /USB3_DM -> Net-(J101-D-)
- J101 pad 3: /USB3_DP -> Net-(J101-D+)
- J201 pad 1: GND -> Net-(J201-Pin_1)
- J301 pad A6: /USB Hub Chip/USBDP -> Net-(D302-I/O2-Pad3)
- J301 pad A7: /USB Hub Chip/USBDM -> Net-(D302-I/O1-Pad1)
- J301 pad B6: /USB Hub Chip/USBDP -> Net-(D302-I/O2-Pad3)
- J301 pad B7: /USB Hub Chip/USBDM -> Net-(D302-I/O1-Pad1)
- J501 pad 1: GND -> /Relay Breakout/RELAY_OUT_1A
- J501 pad 10: +5V -> GND
- J501 pad 11: +5V -> /Relay Breakout/RELAY_OUT_3B
- J501 pad 12: +5V -> +3V3
- J501 pad 13: /Relay Breakout/RELAY_OUT_1A -> /Relay Breakout/RELAY_OUT_4A
- J501 pad 14: /Relay Breakout/RELAY_OUT_1A -> GND
- J501 pad 15: /Relay Breakout/RELAY_OUT_1B -> /Relay Breakout/RELAY_OUT_4B
- J501 pad 16: /Relay Breakout/RELAY_OUT_1B -> +3V3
- J501 pad 17: /Relay Breakout/RELAY_OUT_2A -> /Relay Breakout/RELAY_OUT_5A
- J501 pad 18: /Relay Breakout/RELAY_OUT_2A -> GND
- J501 pad 19: /Relay Breakout/RELAY_OUT_2B -> /Relay Breakout/RELAY_OUT_5B
- J501 pad 20: /Relay Breakout/RELAY_OUT_2B -> +3V3
- J501 pad 21: /Relay Breakout/RELAY_OUT_3A -> /Relay Breakout/RELAY_OUT_6A
- J501 pad 22: /Relay Breakout/RELAY_OUT_3A -> GND
- J501 pad 23: /Relay Breakout/RELAY_OUT_3B -> /Relay Breakout/RELAY_OUT_6B
- J501 pad 24: /Relay Breakout/RELAY_OUT_3B -> +3V3
- J501 pad 25: /Relay Breakout/RELAY_OUT_4A -> /Relay Breakout/RELAY_OUT_7A
- J501 pad 26: /Relay Breakout/RELAY_OUT_4A -> GND
- J501 pad 27: /Relay Breakout/RELAY_OUT_4B -> /Relay Breakout/RELAY_OUT_7B
- J501 pad 28: /Relay Breakout/RELAY_OUT_4B -> +3V3
- J501 pad 3: GND -> /Relay Breakout/RELAY_OUT_1B
- J501 pad 4: GND -> +3V3
- J501 pad 5: +3V3 -> /Relay Breakout/RELAY_OUT_2A
- J501 pad 6: +3V3 -> GND
- J501 pad 7: +3V3 -> /Relay Breakout/RELAY_OUT_2B
- J501 pad 9: +5V -> /Relay Breakout/RELAY_OUT_3A
- R202 pad 1: RP2-USB-DP -> _USB_INFRA_D+
- R203 pad 1: RP2-USB-DM -> _USB_INFRA_D-
- R204 pad 1: +3V3 -> Net-(D203-A)
- R204 pad 2: Net-(Q201-D) -> Net-(U201-GPIO15)
- U201 pad 11: unconnected-(U201-GPIO8-Pad11) -> RELAIS_1
- U201 pad 12: Net-(U201-GPIO9) -> RELAIS_2
- U201 pad 13: Net-(U201-GPIO10) -> RELAIS_3
- U201 pad 14: Net-(U201-GPIO11) -> RELAIS_4
- U201 pad 15: Net-(U201-GPIO12) -> RELAIS_5
- U201 pad 16: Net-(U201-GPIO13) -> RELAIS_6
- U201 pad 17: Net-(U201-GPIO14) -> RELAIS_7
- U201 pad 2: unconnected-(U201-GPIO0-Pad2) -> Net-(J201-Pin_1)
- U201 pad 26: Net-(U201-RUN) -> unconnected-(U201-RUN-Pad26)
- U201 pad 3: RELAIS_1 -> Net-(J201-Pin_2)
- U201 pad 4: RELAIS_2 -> Net-(J201-Pin_3)
- U201 pad 5: RELAIS_3 -> Net-(J201-Pin_4)
- U201 pad 6: RELAIS_4 -> Net-(J201-Pin_5)
- U201 pad 7: RELAIS_5 -> Net-(J201-Pin_6)
- U201 pad 8: RELAIS_6 -> Net-(J201-Pin_7)
- U201 pad 9: RELAIS_7 -> Net-(J201-Pin_8)
- U302 pad 1: RP2-USB-DM -> /USB Hub Chip/USB_DM1
- U302 pad 16: RP2_BOOT -> /USB2_PWR
- U302 pad 2: RP2-USB-DP -> /USB Hub Chip/USB_DP1
- U302 pad 20: /USB4_PWR -> RP2_BOOT
- U302 pad 30: /USB Hub Chip/USBDM -> Net-(U302-USBDM_UP)
- U302 pad 31: /USB Hub Chip/USBDP -> Net-(U302-USBDP_UP)
- U302 pad 6: /USB3_DM -> /USB Hub Chip/USB_DM3
- U302 pad 7: /USB3_DP -> /USB Hub Chip/USB_DP3
- U401 pad 4: /USB1_PWR -> /USB2_PWR
Routing:
- net /USB Power Switch DUT/VOUT: track 41.4 -> 249.0 mm
- net Net-(U201-GPIO24): track 14.5 -> 208.6 mm
- net +3V3: track 199.7 -> 385.9 mm, vias 4 -> 3
- net Net-(U201-GPIO15): track 18.5 -> 204.3 mm
- net GND: track 15.7 -> 187.7 mm, vias 172 -> 155
- net +5V: track 113.1 -> 253.1 mm, vias 2 -> 6
- net Net-(D103-A): track 88.1 -> 2.04 mm, vias 2 -> 0
- net RP2-USB-DP: track 80.9 -> 0.00 mm, vias 2 -> 0
- net RP2-USB-DM: track 79.0 -> 0.00 mm, vias 2 -> 0
- net Net-(D201-A): track 69.2 -> 1.91 mm, vias 2 -> 0
- net Net-(D102-A): track 67.0 -> 0.00 mm, vias 2 -> 0
- net RELAIS_7: track 84.7 -> 22.2 mm
- net /RP2 CPU/12MHz: track 3.39 -> 65.4 mm, vias 0 -> 3
- net RELAIS_6: track 80.1 -> 19.7 mm
- net RELAIS_5: track 75.4 -> 17.0 mm
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Other:
- board size 100 x 160 mm -> 100 x 165 mm
- board text added: "(blue)"
- board text added: "(red)"
- board text added: "1"
- board text added: "11"
- board text added: "12"
- board text added: "13"
- board text added: "14"
- board text added: "15"
- board text added: "16"
- board text added: "17"
- board text added: "18"
- board text added: "19"
- board text added: "2"
- board text added: "21"
- board text added: "22"
- board text added: "23"
- board text added: "24"
- board text added: "25"
- board text added: "26"
- board text added: "27"
- board text added: "28"
- board text added: "29"
- board text added: "3"
- board text added: "31"
- board text added: "32"
- board text added: "33"
- board text added: "34"
- board text added: "35"
- board text added: "36"
- board text added: "37"
- board text added: "38"
- board text added: "39"
- board text added: "4"
- board text added: "5"
- board text added: "6"
- board text added: "7"
- board text added: "8"
- board text added: "9"
- board text added: "Device Under Test Power (green)"
- board text added: "Infra"
- board text added: "Infrastructure (green) Power"
- board text added: "OCTOBUS_"
- board text added: "PICO_INFRA"
- board text added: "PICO_PROBE"
- board text added: "USB Hub"
- board text added: "level shifter"
- board text added: "www.github.com/octoprobe/tentacle"
- board text removed: "3V3"
- board text removed: "5V"
- board text removed: "Reset"
- board text removed: "Tags"

Commit message: Fix D302
Parts:
- removed the Logo_open_hardware101 at (153.2, 50.3)
- moved D302 0.09 mm to (80.2, 27.8)
Connections:
- J301 pad A6: Net-(D302-I/O2-Pad3) -> Net-(D302-I/O1-Pad1)
- J301 pad A7: Net-(D302-I/O1-Pad1) -> Net-(D302-I/O2-Pad3)
- J301 pad B6: Net-(D302-I/O2-Pad3) -> Net-(D302-I/O1-Pad1)
- J301 pad B7: Net-(D302-I/O1-Pad1) -> Net-(D302-I/O2-Pad3)
- NT301 pad 1: Net-(D302-I/O1-Pad1) -> Net-(D302-I/O2-Pad3)
- NT301 pad 3: Net-(D302-I/O2-Pad3) -> Net-(D302-I/O1-Pad1)
Routing:
- net GND: track 187.7 -> 188.6 mm
- net Net-(D302-I/O2-Pad3): track 15.1 -> 15.4 mm, vias 0 -> 3
- net Net-(D302-I/O1-Pad1): track 15.0 -> 15.1 mm, vias 2 -> 0
