File: kicad/tentacle/pcb_octoprobe_usbhubchip.kicad_sch (KiCad schematic)
At the start: 33 parts, among them J301 USB_C_Receptacle_USB2.0, U301 AMS1117-3.3, U302 USB2514B_Bi, Y301 24MHz

Commit message: Tentacle v0.4
Parts:
- added NT301, NT302: octoprobe_NetTie_USB_Differential, 00_project_library:octoprobe_NetTie_USB_Differential, symbol 00_project_library:octoprobe_NetTie_USB_Differential
- C301, C302, C303, C304, C305, C306, C309, C310: JLC (none) -> C1525
- C311, C312: JLC (none) -> C19702
- D301: value LED_PWR (green) -> green; Label (none) -> LED_PWR (green)
- R301: footprint Resistor_SMD:R_0603_1608Metric -> Resistor_SMD:R_0805_2012Metric
Connections:
- removed net USBDM: D302.3 (I/O2), D302.4 (I/O2), J301.A7 (D-), J301.B7 (D-), U302.30 (USBDM_UP)
- removed net USBDP: D302.1 (I/O1), D302.6 (I/O1), J301.A6 (D+), J301.B6 (D+), U302.31 (USBDP_UP)
- new net: NT302.3, U302.30 (USBDM_UP)
- new net: NT302.1, U302.31 (USBDP_UP)
- new net: D302.1 (I/O1), D302.6 (I/O1), J301.A7 (D-), J301.B7 (D-), NT301.1
- new net: D302.3 (I/O2), D302.4 (I/O2), J301.A6 (D+), J301.B6 (D+), NT301.3
- new net USB_UP_D+: NT301.4, NT302.2
- new net USB_UP_D-: NT301.2, NT302.4

Commit message: Fix D302
Connections:
- net at J301.A7 (D-), J301.B7 (D-), NT301.1: now also D302.3 (I/O2), D302.4 (I/O2); no longer D302.1 (I/O1), D302.6 (I/O1)
- net at J301.A6 (D+), J301.B6 (D+), NT301.3: now also D302.1 (I/O1), D302.6 (I/O1); no longer D302.3 (I/O2), D302.4 (I/O2)
Changed lines of the file:
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@@
-	)
-	(junction
-		(at 67.31 48.26)
-		(diameter 0)
-		(color 0 0 0 0)
 	)
 	(junction
@@
 	(junction
 		(at 97.79 125.73)
-		(diameter 0)
-		(color 0 0 0 0)
-	)
-	(junction
-		(at 92.71 50.8)
 		(diameter 0)
 		(color 0 0 0 0)
@@
 	)
 	(junction
+		(at 92.71 48.26)
+		(diameter 0)
+		(color 0 0 0 0)
+	)
+	(junction
 		(at 92.71 64.77)
 		(diameter 0)
@@
 	)
 	(junction
+		(at 67.31 50.8)
+		(diameter 0)
+		(color 0 0 0 0)
+	)
+	(junction
+		(at 207.01 38.1)
+		(diameter 0)
+		(color 0 0 0 0)
+	)
+	(junction
+		(at 41.91 172.72)
+		(diameter 0)
+		(color 0 0 0 0)
+	)
+	(junction
+		(at 208.28 153.67)
+		(diameter 0)
+		(color 0 0 0 0)
+	)
+	(junction
+		(at 195.58 143.51)
+		(diameter 0)
+		(color 0 0 0 0)
+	)
+	(junction
+		(at 34.29 71.12)
+		(diameter 0)
+		(color 0 0 0 0)
+	)
+	(junction
+		(at 204.47 38.1)
+		(diameter 0)
+		(color 0 0 0 0)
+	)
+	(junction
+		(at 91.44 125.73)
+		(diameter 0)
+		(color 0 0 0 0)
+	)
+	(junction
 		(at 67.31 64.77)
-		(diameter 0)
-		(color 0 0 0 0)
-	)
-	(junction
-		(at 207.01 38.1)
-		(diameter 0)
-		(color 0 0 0 0)
-	)
-	(junction
-		(at 41.91 172.72)
-		(diameter 0)
-		(color 0 0 0 0)
-	)
-	(junction
-		(at 208.28 153.67)
-		(diameter 0)
-		(color 0 0 0 0)
-	)
-	(junction
-		(at 195.58 143.51)
-		(diameter 0)
-		(color 0 0 0 0)
-	)
-	(junction
-		(at 34.29 71.12)
-		(diameter 0)
-		(color 0 0 0 0)
-	)
-	(junction
-		(at 204.47 38.1)
-		(diameter 0)
-		(color 0 0 0 0)
-	)
-	(junction
-		(at 91.44 125.73)
 		(diameter 0)
 		(color 0 0 0 0)
@@
 	(wire
 		(pts
+			(xy 92.71 48.26) (xy 92.71 64.77)
+		)
+		(stroke
+			(width 0)
+			(type default)
+		)
+	)
+	(wire
+		(pts
 			(xy 80.01 33.02) (xy 92.71 33.02)
 		)
@@
 	(wire
 		(pts
-			(xy 50.8 50.8) (xy 92.71 50.8)
+			(xy 50.8 50.8) (xy 67.31 50.8)
 		)
 		(stroke
@@
 	(wire
 		(pts
-			(xy 67.31 48.26) (xy 97.79 48.26)
-		)
-		(stroke
-			(width 0)
-			(type solid)
-		)
-	)
-	(wire
-		(pts
 			(xy 180.34 106.68) (xy 180.34 104.14)
 		)
@@
 	(wire
 		(pts
+			(xy 67.31 50.8) (xy 67.31 64.77)
+		)
+		(stroke
+			(width 0)
+			(type default)
+		)
+	)
+	(wire
+		(pts
 			(xy 59.69 40.64) (xy 63.5 40.64)
 		)
@@
 	(wire
 		(pts
-			(xy 92.71 50.8) (xy 97.79 50.8)
-		)
-		(stroke
-			(width 0)
-			(type solid)
-		)
-	)
-	(wire
-		(pts
 			(xy 208.28 151.13) (xy 208.28 153.67)
 		)
@@
 	(wire
 		(pts
-			(xy 67.31 48.26) (xy 67.31 64.77)
-		)
-		(stroke
-			(width 0)
-			(type default)
-		)
-	)
-	(wire
-		(pts
 			(xy 209.55 38.1) (xy 212.09 38.1)
 		)
@@
 	(wire
 		(pts
-			(xy 92.71 50.8) (xy 92.71 64.77)
-		)
-		(stroke
-			(width 0)
-			(type default)
-		)
-	)
-	(wire
-		(pts
 			(xy 254 35.56) (xy 254 38.1)
 		)
@@
 	(wire
 		(pts
+			(xy 92.71 48.26) (xy 97.79 48.26)
+		)
+		(stroke
+			(width 0)
+			(type solid)
+		)
+	)
+	(wire
+		(pts
 			(xy 222.25 143.51) (xy 222.25 144.78)
 		)
@@
 	(wire
 		(pts
+			(xy 67.31 50.8) (xy 97.79 50.8)
+		)
+		(stroke
+			(width 0)
+			(type solid)
+		)
+	)
+	(wire
+		(pts
 			(xy 67.31 68.58) (xy 68.58 68.58)
 		)
@@
 	(wire
 		(pts
-			(xy 50.8 48.26) (xy 67.31 48.26)
-		)
-		(stroke
+			(xy 50.8 48.26) (xy 92.71 48.26)
+		)
+		(stroke
