File: kicad/tentacle_v0.7/pcb_tentacle.kicad_pcb (KiCad board)
At the start: 2 copper layers, 100 x 165 mm, 961 parts, among them J1302 Conn_02x20, J1303 Conn_02x20, J1501 Conn_02x20, J1502 Conn_01x12, J201 Conn_02x05, J202 Conn_01x5, J301 USB_C_Receptacle_USB2.0, J501 Conn_02x20, U1001 GAQY221S, U1101 GAQY221S, U1201 GAQY221S, U1501 RP2040, U1502 W25Q32JVS, U1503 TXB0108PW, U1504 TXB0108PW, U201 RP2040, U202 AMS1117-3.3, U203 W25Q32JVS, U204 TPS2595xx, U205 TPS2595xx, U207 TPS2595xx, U302 USB2514B_Bi, U601 GAQY221S, U701 GAQY221S, U801 GAQY221S, U901 GAQY221S, X201 Oscillator-12MHz, Y301 24MHz

Commit message: Tenatcle: v0.7. Manually fix all violations.
Routing:
- net Net-(J201-Pin_8): track 60.3 -> 50.6 mm
- net +5Vbuf: track 113.0 -> 115.1 mm
- net GND: track 161.3 -> 162.3 mm, vias 477 -> 453
- net /RP2 PROBE/GPIO18: track 28.3 -> 27.3 mm
- net /RP2 PROBE/+1V1: track 27.1 -> 27.9 mm
- net /RP2 PROBE/QSPI_SCLK: track 14.3 -> 15.0 mm
- net /RP2 CPU/12MHz: track 58.7 -> 58.1 mm
- net /RP2 PROBE/GPIO27: track 37.5 -> 36.9 mm
- net Net-(J201-Pin_5): track 43.8 -> 43.3 mm
- net /RP2 PROBE/GPIO22: track 34.0 -> 33.5 mm
- net (no net): vias 2 -> 1

Commit message: Tentacle: v0.7.1
Parts:
- R311: value 10k -> 100k
Connections:
- R311 pad 1: +3V3 -> GND
Routing:
- net +3V3: track 91.9 -> 89.6 mm
- net GND: track 162.3 -> 161.6 mm
Changed lines of the file:
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@@
 	(title_block
 		(title "Octoprobe Tentacle")
-		(date "2026-01-20")
-		(rev "0.7")
+		(date "2026-02-18")
+		(rev "0.7.1")
 		(company "Hans Märki, Märki Informatik")
 		(comment 1 "The MIT License (MIT)")
@@
 			)
 		)
-		(fp_text user "5"
+		(fp_text user "16"
 			(at -5.334 5.08 90)
 			(unlocked yes)
@@
 			)
 		)
-		(fp_text user "0"
+		(fp_text user "10"
 			(at 2.794 0 90)
 			(unlocked yes)
@@
 			)
 		)
-		(fp_text user "2"
+		(fp_text user "11"
 			(at 2.794 2.794 90)
 			(unlocked yes)
@@
 			)
 		)
-		(fp_text user "7"
+		(fp_text user "17"
 			(at -5.334 7.874 90)
 			(unlocked yes)
@@
 			)
 		)
-		(fp_text user "3"
+		(fp_text user "15"
 			(at -5.334 2.54 90)
 			(unlocked yes)
@@
 			)
 		)
-		(fp_text user "1"
+		(fp_text user "14"
 			(at -5.334 0 90)
 			(unlocked yes)
@@
 			)
 		)
-		(fp_text user "8"
+		(fp_text user "13"
 			(at 2.794 7.62 90)
 			(unlocked yes)
@@
 			)
 		)
-		(fp_text user "4"
+		(fp_text user "12"
 			(at 2.794 5.08 90)
 			(unlocked yes)
@@
 			)
 		)
-		(fp_text user "2"
+		(fp_text user "11"
 			(at 2.814 2.794 90)
 			(unlocked yes)
@@
 			)
 		)
-		(fp_text user "1"
+		(fp_text user "14"
 			(at -5.314 0 90)
 			(unlocked yes)
@@
 			)
 		)
-		(fp_text user "4"
+		(fp_text user "12"
 			(at 2.814 5.08 90)
 			(unlocked yes)
@@
 			)
 		)
-		(fp_text user "3"
+		(fp_text user "15"
 			(at -5.314 2.54 90)
 			(unlocked yes)
@@
 			)
 		)
-		(fp_text user "7"
+		(fp_text user "17"
 			(at -5.314 7.874 90)
 			(unlocked yes)
@@
 			)
 		)
-		(fp_text user "8"
+		(fp_text user "13"
 			(at 2.814 7.62 90)
 			(unlocked yes)
@@
 			)
 		)
-		(fp_text user "5"
+		(fp_text user "16"
 			(at -5.314 5.08 90)
 			(unlocked yes)
@@
 			)
 		)
-		(fp_text user "0"
+		(fp_text user "10"
 			(at 2.814 0 90)
 			(unlocked yes)
@@
 			)
 		)
-		(property "Value" "10k"
+		(property "Value" "100k"
 			(at 0 1.17 90)
 			(layer "F.Fab")
@@
 			(layers "F.Cu" "F.Mask" "F.Paste")
 			(roundrect_rratio 0.25)
-			(net 12 "+3V3")
+			(net 5 "GND")
 			(pintype "passive")
 		)
@@
 	)
 	(segment
-		(start 117.3142 23.3472)
-		(end 117.3142 22.6758)
-		(width 0.15)
-		(layer "F.Cu")
-		(net 5)
-	)
-	(segment
 		(start 66.4585 177.923)
 		(end 66.4585 176.5675)
@@
 	)
 	(via
-		(at 117.3142 22.75)
+		(at 117.31 22.46)
 		(size 0.45)
 		(drill 0.3)
@@
 	)
 	(segment
-		(start 116.97 22.2)
-		(end 116.38 22.79)
-		(width 0.2)
-		(layer "F.Cu")
-		(net 12)
-	)
-	(segment
 		(start 123.9386 29.6806)
 		(end 123.3812 29.6806)
@@
 	)
 	(segment
-		(start 116.38 22.79)
-		(end 116.38 23.3162)
-		(width 0.2)
-		(layer "F.Cu")
-		(net 12)
-	)
-	(segment
 		(start 117.365 25.257401)
 		(end 117.8842 24.738201)
@@
 		(width 0.2)
 		(layer "F.Cu")
-		(net 12)
-	)
-	(segment
-		(start 117.8842 22.2)
-		(end 116.97 22.2)
-		(width 0.2)
-		(layer "F.Cu")
