File: kicad/tentacle_v0.7/pcb_tentacle.kicad_sch (KiCad schematic)
At the start: 10 parts, among them J202 Conn_01x5

Commit message: Tentacle v0.7: Fix LEDs. Import new symbols and footprints
Parts:
- D101: footprint 00_project_library:LED_0603_1608Metric -> LED_SMD:LED_0805_2012Metric; JLC C2290 -> C34499
Changed lines of the file:
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@@
 			)
 		)
-		(property "Footprint" "00_project_library:LED_0603_1608Metric"
+		(property "Footprint" "LED_SMD:LED_0805_2012Metric"
 			(at 109.22 67.31 0)
 			(effects
@@
 			)
 		)
-		(property "Description" ""
+		(property "Description" "Light emitting diode"
 			(at 109.22 67.31 0)
 			(effects
@@
 			)
 		)
-		(property "JLC" "C2290"
+		(property "JLC" "C34499"
 			(at 109.22 67.31 0)
 			(effects

Commit message: Tentacle: v0.7
Parts:
- added BP220: USB_PROBE_D-, 00_project_library:octoprobe_breakout_PB, symbol 00_project_library:octoprobe_breakout_BP
- added BP221: USB_PROBE_D+, 00_project_library:octoprobe_breakout_PB, symbol 00_project_library:octoprobe_breakout_BP
- added BP222: USB_PROBE_PWR, 00_project_library:octoprobe_breakout_PB, symbol 00_project_library:octoprobe_breakout_BP
- added BP223: USB_PROBE_5V, 00_project_library:octoprobe_breakout_PB, symbol 00_project_library:octoprobe_breakout_BP
- added BP224: USB_PROBE_GND, 00_project_library:octoprobe_breakout_PB, symbol 00_project_library:octoprobe_breakout_BP
- added R220, R221: 0R, Resistor_SMD:R_0603_1608Metric, symbol Device:R
Connections:
- net GND: now also BP224.1
- net USB Hub Chip/PRT_PWR4: now also BP222.1
- net _USB_PROBE_D+: now also R221.1; no longer NT102.3
- net _USB_PROBE_D-: now also R220.1; no longer NT102.1
- new net: BP220.1, NT102.1, R220.2
- new net: BP221.1, NT102.3, R221.2
- new net +5Vbuf: BP223.1
- no-connect marks 4 -> 3
