File: kicad/tentacle_v0.7/pcb_tentacle_opto_relay.kicad_sch (KiCad schematic)
At the start: 5 parts, among them U601 GAQY221S

Commit message: Tentacle v0.7: Fix LEDs. Import new symbols and footprints
Parts:
- D601: footprint 00_project_library:LED_0603_1608Metric -> LED_SMD:LED_0805_2012Metric; JLC C2290 -> C34499
Changed lines of the file:
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@@
 			)
 		)
-		(property "Footprint" "00_project_library:LED_0603_1608Metric"
+		(property "Footprint" "LED_SMD:LED_0805_2012Metric"
 			(at 100.33 49.53 0)
 			(effects
@@
 			)
 		)
-		(property "Description" ""
+		(property "Description" "Light emitting diode"
 			(at 100.33 49.53 0)
 			(effects
@@
 			)
 		)
-		(property "JLC" "C2290"
+		(property "JLC" "C34499"
 			(at 100.33 49.53 0)
 			(effects
